File: aether/aether.kicad_sch (KiCad schematic)
At the start: 0 parts

Commit message: sch: start lora module
Parts:
- added AE1: Antenna, symbol Device:Antenna
- added D1: 3.0V, symbol Device:D_Zener
- added R1: 36k, symbol Device:R
- added U1: LoRa-E5, symbol LoRa-E5:LoRa-E5
Connections:
- new net: D1.1 (K), R1.2, U1.8 (PB3)
- new net: AE1.1 (A), U1.15 (RFIO)
- new net GND: D1.2 (A), U1.14 (GND), U1.16 (GND), U1.2 (GND), U1.22 (GND)
- new net USB5V: R1.1
- new net VCC: U1.1 (VCC)
Other:
- note added: "Detect USB and wake up"
- company: (none) -> University of Central Florida
- title: (none) -> Aether Sensor Network - LoRa Module
