File: subsheets/mcu.kicad_sch (KiCad schematic)
At the start: 25 parts, among them J2 Conn_01x05, U5 LoRa-E5

Commit message: -
-
Parts:
- removed D5: 3.0V, Diode_SMD:D_0805_2012Metric_Pad1.15x1.40mm_HandSolder, symbol Device:D_Zener
- added R27: 68K, Resistor_SMD:R_0805_2012Metric_Pad1.20x1.40mm_HandSolder, symbol Device:R_US
Connections:
- net GND: now also R27.1
- net PB3: now also R27.2
Changed lines of the file:
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@@
   (junction (at 96.52 58.42) (diameter 0) (color 0 0 0 0)
-  )
-  (junction (at 151.13 166.37) (diameter 0) (color 0 0 0 0)
   )
   (junction (at 44.45 36.83) (diameter 0) (color 0 0 0 0)
@@
   (symbol (lib_id "power:GND") (at 236.22 72.39 0) (unit 1)
     (in_bom yes) (on_board yes) (fields_autoplaced)
-    (property "Reference" "#PWR043" (id 0) (at 236.22 78.74 0)
+    (property "Reference" "#PWR044" (id 0) (at 236.22 78.74 0)
       (effects (font (size 1.27 1.27)) hide)
     )
@@
   (symbol (lib_id "power:GND") (at 146.05 88.265 0) (unit 1)
     (in_bom yes) (on_board yes) (fields_autoplaced)
-    (property "Reference" "#PWR039" (id 0) (at 146.05 94.615 0)
+    (property "Reference" "#PWR038" (id 0) (at 146.05 94.615 0)
       (effects (font (size 1.27 1.27)) hide)
     )
@@
   (symbol (lib_id "power:GND") (at 151.13 177.8 0) (unit 1)
     (in_bom yes) (on_board yes) (fields_autoplaced)
-    (property "Reference" "#PWR041" (id 0) (at 151.13 184.15 0)
+    (property "Reference" "#PWR040" (id 0) (at 151.13 184.15 0)
       (effects (font (size 1.27 1.27)) hide)
     )
@@
   (symbol (lib_id "power:GND") (at 160.02 68.58 90) (unit 1)
     (in_bom yes) (on_board yes) (fields_autoplaced)
-    (property "Reference" "#PWR042" (id 0) (at 166.37 68.58 0)
+    (property "Reference" "#PWR043" (id 0) (at 166.37 68.58 0)
       (effects (font (size 1.27 1.27)) hide)
     )
@@
   (symbol (lib_id "power:GND") (at 147.32 44.45 90) (unit 1)
     (in_bom yes) (on_board yes)
-    (property "Reference" "#PWR040" (id 0) (at 153.67 44.45 0)
+    (property "Reference" "#PWR039" (id 0) (at 153.67 44.45 0)
       (effects (font (size 1.27 1.27)) hide)
     )
@@
     (pin "1")
   )
-  (symbol (lib_id "Device:D_Zener") (at 151.13 170.18 270) (unit 1)
-    (in_bom yes) (on_board yes) (fields_autoplaced)
-    (property "Reference" "D5" (id 0) (at 153.162 169.2715 90)
-      (effects (font (size 1.27 1.27)) (justify left))
-    )
-    (property "Value" "3.0V" (id 1) (at 153.162 172.0466 90)
-      (effects (font (size 1.27 1.27)) (justify left))
-    )
-    (property "Footprint" "Diode_SMD:D_0805_2012Metric_Pad1.15x1.40mm_HandSolder" (id 2) (at 151.13 170.18 0)
-      (effects (font (size 1.27 1.27)) hide)
-    )
-    (property "Datasheet" "~" (id 3) (at 151.13 170.18 0)
-      (effects (font (size 1.27 1.27)) hide)
-    )
-    (pin "1")
-    (pin "2")
-  )
   (symbol (lib_id "power:GND") (at 153.67 149.86 90) (unit 1)
     (in_bom yes) (on_board yes)
-    (property "Reference" "#PWR0101" (id 0) (at 160.02 149.86 0)
+    (property "Reference" "#PWR042" (id 0) (at 160.02 149.86 0)
       (effects (font (size 1.27 1.27)) hide)
     )
@@
   (symbol (lib_id "power:GND") (at 153.67 143.51 90) (unit 1)
     (in_bom yes) (on_board yes)
-    (property "Reference" "#PWR038" (id 0) (at 160.02 143.51 0)
+    (property "Reference" "#PWR041" (id 0) (at 160.02 143.51 0)
       (effects (font (size 1.27 1.27)) hide)
     )
@@
     (pin "8")
   )
+  (symbol (lib_id "Device:R_US") (at 151.13 170.18 180) (unit 1)
+    (in_bom yes) (on_board yes) (fields_autoplaced)
+    (property "Reference" "R27" (id 0) (at 152.781 169.2715 0)
+      (effects (font (size 1.27 1.27)) (justify right))
+    )
+    (property "Value" "68K" (id 1) (at 152.781 172.0466 0)
+      (effects (font (size 1.27 1.27)) (justify right))
+    )
+    (property "Footprint" "Resistor_SMD:R_0805_2012Metric_Pad1.20x1.40mm_HandSolder" (id 2) (at 150.114 169.926 90)
+      (effects (font (size 1.27 1.27)) hide)
+    )
+    (property "Datasheet" "~" (id 3) (at 151.13 170.18 0)
+      (effects (font (size 1.27 1.27)) hide)
+    )
+    (pin "1")
+    (pin "2")
+  )
   (symbol (lib_id "Device:R_US") (at 85.09 46.99 0) (unit 1)

Commit message: Updated Schematics
-
Connections:
- net +3.3V: no longer R22.1, R23.1
- net +5V: now also R22.1, R23.1
Other:
- moved on the sheet: H1, H2, H3, H4, J2, R26, R27, S1

Commit message: Final Schematic
-
Other:
- note added: "BME688 Sensor"
- note added: "MCU Circuit"
- note added: "Particulate Matter Sensor"
- note added: "ZMOD4510 Sensor"
- moved on the sheet: AE1, BME1, C13, C14, C15, C16, H1, H2, H3, H4, J2, PMSensor1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
